Commit message: Add the two 1-inch swivel casters
Each caster is a swivel joint plus a wheel joint. The wheel trails 10 mm
behind its pivot and swings round as the robot drives. The stability
check now uses the casters' real contact points, so the braking limit
changes with the casters: 0.13 g after driving forward with 250 g in each
outstretched hand, and 0.25 g after reversing.

Co-Authored-By: Claude Opus 5.5 <noreply@anthropic.com>

File: gerdoo.urdf (robot description, URDF)
Before this commit: robot gerdoo, 44 links, 43 joints
Links:
- added link caster_back_swivel; visual box size=0.018 0.0016 0.018; visual box size=0.018 0.0016 0.018
- added link caster_back_wheel; visual box size=0.01875 0.0104 0.0022; visual cylinder length=0.01 radius=0.0125
- added link caster_front_swivel; visual box size=0.018 0.0016 0.018; visual box size=0.018 0.0016 0.018
- added link caster_front_wheel; visual box size=0.01875 0.0104 0.0022; visual cylinder length=0.01 radius=0.0125
Joints:
- added joint caster_back_swivel: type continuous, parent base_link, child caster_back_swivel, origin xyz=-0.09 0 0.0365 rpy=0 0 0, axis 0 0 1
- added joint caster_back_wheel: type continuous, parent caster_back_swivel, child caster_back_wheel, origin xyz=-0.01 0 -0.024 rpy=0 0 0, axis 0 1 0
- added joint caster_front_swivel: type continuous, parent base_link, child caster_front_swivel, origin xyz=0.09 0 0.0365 rpy=0 0 0, axis 0 0 1
- added joint caster_front_wheel: type continuous, parent caster_front_swivel, child caster_front_wheel, origin xyz=-0.01 0 -0.024 rpy=0 0 0, axis 0 1 0

Commit message: Turn the arm mounts 70 degrees outward
J1 = 0 now points 70 deg outward, and the arms face forward at J1 = -70
(left) and +70 (right). The J1 housings turn 70 deg about J1 on their
discs, with a support lobe under each. The whole +/-89 deg J1 range now
clears the body. Also: USB hub holes on the vendor's 58 x 49, 1.5 mm
dock plates, and no light-dial hole on the back cover.

Co-Authored-By: Claude Opus 5.5 <noreply@anthropic.com>

File: gerdoo.urdf (robot description, URDF)
Before this commit: robot gerdoo, 48 links, 47 joints
Joints:
- joint L_mount: origin xyz=-0.04249 0.14568 0.1043 rpy=0 0 -1.570796 -> xyz=-0.0145324 0.105752 0.1043 rpy=0 0 -0.349066
- joint R_mount: origin xyz=-0.04249 -0.14568 0.1043 rpy=0 0 -1.570796 -> xyz=-0.0145324 -0.105752 0.1043 rpy=0 0 -2.792527

Commit message: New neck on two STS3215s, lidar raised 45 mm, dock sign raised to match
- Neck v1: the pan servo stands on the 3rd floor, and the tilt servo lies
  centred under the screen's board bracket, driven from both sides by a
  printed yoke. Joints sit on the real axes: pan +-90 deg, tilt 15 deg down
  to 30 deg up. The face texture follows the new screen position.
- The C1 now sits on lidar-holder-v2, 45 mm higher (scan plane ~349 mm above
  the deck top), and the dock's sign and its light are raised to match.
- Body mass and centre of gravity updated (+150 g, CoG +9 mm).

Co-Authored-By: Claude Opus 5.5 <noreply@anthropic.com>

File: gerdoo.urdf (robot description, URDF)
Before this commit: robot gerdoo, 48 links, 47 joints
Joints:
- joint lidar: origin xyz=0 0 0.3407 rpy=0 0 0 -> xyz=0 0 0.3857 rpy=0 0 0
- joint neck_pan: origin xyz=0.065 0.0005 0.2697 rpy=0 0 0 -> xyz=0.095 0 0.2759 rpy=0 0 0
- joint neck_tilt: limit lower=-0.5236 upper=0.5236 effort=1 velocity=5 -> lower=-0.2618 upper=0.5236 effort=1 velocity=5; origin xyz=0.012 0 0.012 rpy=0 0 0 -> xyz=-0.0005 0 0.0268 rpy=0 0 0

Commit message: Idle pose as the startup pose; pan servo lifted for its cable
- New "Idle" preset (the user's pose: arms folded down beside the body,
  J1 -73, J2 52, J3 33, J4 -9, J5 135, J6 101, J7 81 deg, gripper 74 %),
  mirrored onto the right arm. The page now starts in it. No contacts, lidar
  clear, and a lower centre of gravity than Rest (braking limit 0.42 g).
- Neck: the pan servo sits 8.5 mm higher so its bottom cable sockets have
  room, and the arm's plate now carries the tilt servo directly.

Co-Authored-By: Claude Opus 5.5 <noreply@anthropic.com>

File: gerdoo.urdf (robot description, URDF)
Before this commit: robot gerdoo, 48 links, 47 joints
Joints:
- joint neck_pan: origin xyz=0.095 0 0.2759 rpy=0 0 0 -> xyz=0.095 0 0.2844 rpy=0 0 0
- joint neck_tilt: origin xyz=-0.0005 0 0.0268 rpy=0 0 0 -> xyz=-0.0005 0 0.0183 rpy=0 0 0
